File: CAD/mouse_kicad_rev2/rezq_rev2.kicad_pcb (KiCad board)
At the start: 2 copper layers, 92.8 x 94.6 mm, 99 parts, among them J2 SWD Header, M1 M1_Conn_Alt, M2 M2_Conn_Alt, Q0 TEFT4300, Q1 TEFT4300, Q10 Q_NMOS_GSD, Q11 Q_NMOS_GSD, Q12 Q_NMOS_GSD, Q2 TEFT4300, Q3 TEFT4300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

Commit message: Version 3 PCB and some initial test code
Parts:
- renumbered GND to TP2, +5V to TP3, +3v3V to TP4, GND to TP5, GND to TP6
Connections:
- U7 pad 10: unconnected-(U7-PA0-Pad10) -> M1_SPD
- U7 pad 30: USART1_TX -> unconnected-(U7-PA9-Pad30)
- U7 pad 31: USART1_RX -> unconnected-(U7-PA10-Pad31)
- U7 pad 39: SWO -> unconnected-(U7-PB3-Pad39)
- U7 pad 4: M1_SPD -> unconnected-(U7-PC15-Pad4)
Routing:
- net M1_SPD: track 23.6 -> 26.8 mm
