File: CAD/mouse2_kicad_rev1/mouse2_rev1.kicad_sch (KiCad schematic)
At the start: 121 parts, among them IC1 STM32F405RGT6, J1 SWD Header, J2 SWD Header, M1 M1_Conn_Alt, M2 M2_Conn_Alt, Q0 TEFT4300, Q1 TEFT4300, Q10 Q_NMOS_GSD, Q11 Q_NMOS_GSD, Q12 Q_NMOS_GSD, Q2 TEFT4300, Q3 TEFT4300, Q9 Q_NMOS_GSD, SW1 SW, SW2 SW, SW3 SW, U1 PMW3389DM-T3QU, U10 TPS7A2033PDBVR, U11 LM66100DCKR, U2 L293D, U3 TLV70019_SOT23-5, U4 BC832, U5 LM66100DCKR, U6 LM66100DCKR, U7 ICM-45605, U8 TPS7A2033PDBVR, U9 TS30011-M050QFNR, Y1 ABS07-32.768KHZ-T

Commit message: Mouse 2 is ballin ish! got a bunch of layout done
Parts:
- removed C38: 22uF, Capacitor_SMD:C_0805_2012Metric_Pad1.18x1.45mm_HandSolder, symbol Device:C
- removed C40: 0.1uF, Capacitor_SMD:C_0805_2012Metric_Pad1.18x1.45mm_HandSolder, symbol Device:C
- removed MOS1: SSM3K335R_LF, custom_foot:SOT-23F_TOS, symbol SSM3K3335R:SSM3K335R_LF
- removed R13, R14, R15, R16: 47k, Resistor_SMD:R_1206_3216Metric_Pad1.30x1.75mm_HandSolder, symbol bloo-rescue:R-Device-mouse_v2-rescue
- removed R5, R6, R7, R8: 35, Resistor_SMD:R_1206_3216Metric_Pad1.30x1.75mm_HandSolder, symbol bloo-rescue:R-Device-mouse_v2-rescue
- removed RST1, SW1, SW2, SW3: SW, Button_Switch_SMD:SW_SPST_REED_CT05-XXXX-G1, symbol Switch:SW_Push
- removed U6: LM66100DCKR, custom_foot:DCK6_TEX, symbol DCK6_TEX:LM66100DCKR
- added C22: 15pF, Capacitor_SMD:C_0603_1608Metric_Pad1.08x0.95mm_HandSolder, symbol Device:C
- added C25: 0.1uF, Capacitor_SMD:C_0603_1608Metric_Pad1.08x0.95mm_HandSolder, symbol Device:C
- added C26: 10uF, Capacitor_SMD:C_0603_1608Metric_Pad1.08x0.95mm_HandSolder, symbol Device:C
- added R13, R14, R15, R28: 47K, Resistor_SMD:R_0603_1608Metric_Pad0.98x0.95mm_HandSolder, symbol Device:R
- added R16: 10k, Resistor_SMD:R_0603_1608Metric_Pad0.98x0.95mm_HandSolder, symbol Device:R
- added R5, R6, R7, R8: 35, Resistor_SMD:R_0603_1608Metric_Pad0.98x0.95mm_HandSolder, symbol Device:R
- added S1, S3, S4, S6: SKRPABE010, BUTTON:SW_SKRPABE010, symbol BUTTON:SKRPABE010
- added Y2: 16MHz, Crystal:Crystal_SMD_2016-4Pin_2.0x1.6mm, symbol UCIRP-KiCAD-Lib:Crystal_GND24_Small
- C14, C15, C18, C20, C24, C27, C28, C29, C3, C30, C31, C32, C33, C34, C39, C8: footprint Capacitor_SMD:C_1206_3216Metric_Pad1.33x1.80mm_HandSolder -> Capacitor_SMD:C_0603_1608Metric_Pad1.08x0.95mm_HandSolder
- C19: value 0.1uF -> 10uF; footprint Capacitor_SMD:C_1206_3216Metric_Pad1.33x1.80mm_HandSolder -> Capacitor_SMD:C_0603_1608Metric_Pad1.08x0.95mm_HandSolder
- C21: value 1uF -> 0.1uF; footprint Capacitor_SMD:C_1206_3216Metric_Pad1.33x1.80mm_HandSolder -> Capacitor_SMD:C_0603_1608Metric_Pad1.08x0.95mm_HandSolder
- C23: value 15pF -> 22uF; footprint Capacitor_SMD:C_1206_3216Metric_Pad1.33x1.80mm_HandSolder -> Capacitor_SMD:C_0603_1608Metric_Pad1.08x0.95mm_HandSolder
- C35, C36: value 10uF -> 0.1uF; footprint Capacitor_SMD:C_1206_3216Metric_Pad1.33x1.80mm_HandSolder -> Capacitor_SMD:C_0603_1608Metric_Pad1.08x0.95mm_HandSolder
- C37: footprint Capacitor_SMD:C_0805_2012Metric_Pad1.18x1.45mm_HandSolder -> Capacitor_SMD:C_0603_1608Metric_Pad1.08x0.95mm_HandSolder
- C4: value 0.1uF -> 1uF; footprint Capacitor_SMD:C_1206_3216Metric_Pad1.33x1.80mm_HandSolder -> Capacitor_SMD:C_0603_1608Metric_Pad1.08x0.95mm_HandSolder
- R1, R11, R12, R19, R2, R20, R21, R23, R24, R25, R26, R3, R4, R9: footprint Resistor_SMD:R_1206_3216Metric_Pad1.30x1.75mm_HandSolder -> Resistor_SMD:R_0603_1608Metric_Pad0.98x0.95mm_HandSolder
- R17, R27: value 10K -> 10k; footprint Resistor_SMD:R_1206_3216Metric_Pad1.30x1.75mm_HandSolder -> Resistor_SMD:R_0603_1608Metric_Pad0.98x0.95mm_HandSolder
- R18: value 20K -> 20k; footprint Resistor_SMD:R_1206_3216Metric_Pad1.30x1.75mm_HandSolder -> Resistor_SMD:R_0603_1608Metric_Pad0.98x0.95mm_HandSolder
- U1: footprint (none) -> PMW3389:PMW3360DM
- Y1: footprint ABS07-32.768KHZ-T:XTAL_ABS07-32.768KHZ-T -> AS07-XTAL:XTAL_ABS07-32.768KHZ-T
Connections:
- net +5V_NET is gone; now on net +5V: C37.1, L2.2, U11.3 (*CE), U5.3 (*CE), U9.5 (FB)
- net VSS is gone; now on net GND: IC1.18 (VSS_1), IC1.63 (VSS_2)
- net VSSA is gone; now on net GND: IC1.12 (VSSA)
- net +1V9: no longer C1.1, C11.1, C18.1, C27.1, C28.1, C29.1, C30.1, C32.1, C43.1, C6.1, C8.1, IC1.1 (VBAT), IC1.19 (VDD_1), IC1.32 (VDD_2), IC1.48 (VDD_3), IC1.64 (VDD_4), M1.3 (Pin_3), M2.3 (Pin_3), R10.1, R11.1, R12.2, R19.2, R20.2, R21.2, R23.1, R24.1, R25.1, R26.2, R9.1, U1.5 (VDDIO), U3.1 (IN), U3.3 (EN), U4.16 (VDD), U5.6 (VOUT), U8.5 (OUT)
- net +3V3A: now also C19.1, C31.2, C4.1, IC1.13 (VDDA); no longer C21.1, C7.1, U7.5 (VDDIO)
- net +5V: now also C23.1, C35.2; no longer C4.1
- net BC_RST: now also R25.1; no longer R25.2
- net BOOT0: now also R17.1; no longer R17.2
- net BUTTON: now also S4.1, S4.2
- net BUTTON_2: now also R28.2, S3.1, S3.2; no longer R24.2
- net BUTTON_3: now also S1.1, S1.2
- net EMIT_1: now also R24.1
- net EMIT_2: now also R13.1
- net EMIT_3: now also R14.1
- net EMIT_4: now also R15.1
- net GND: now also C1.2, C10.2, C11.2, C12.2, C13.2, C14.2, C15.2, C16.2, C17.2, C18.2, C2.2, C20.2, C21.1, C27.1, C28.1, C29.1, C31.1, C32.1, C35.1, C36.2, C44.2, C5.2, C6.2, C7.2, C8.1, C9.2, R1.1, R17.2, R2.1, R24.2, R3.1, R4.1, U1.8 (GND), U10.2 (GND), U3.2 (GND), U7.6 (GND), C22.2, R13.2, R14.2, R15.2, S1.3, S1.4, S3.3, S3.4, S4.3, S4.4, S6.3, S6.4, Y2.2; no longer C23.2, C27.2, C28.2, C29.2, C31.2, C32.2, C35.2, C8.2, R17.1
- net IMU_POCI: now also R16.2
- net MOUSE_CS: now also IC1.50 (PA15)
- net MOUSE_PICO: now also IC1.53 (PC12)
- net MOUSE_POCI: now also IC1.56 (PB4)
- net MOUSE_SCLK: now also IC1.55 (PB3)
- net PGND: now also C23.2, NT2.2, C25.1, C26.2; no longer C36.2
- net VCC: now also S2.2, U9.11 (VCC), U9.2 (VCC), U9.3 (VCC), C25.2, C26.1
- net at D3.1 (K): now also R8.1
- net at Q12.3 (D): now also R8.2
- net at D2.1 (K): now also R7.1
- net at Q11.3 (D): now also R7.2
- net at D0.1 (K): now also R5.1
- net at Q9.3 (D): now also R5.2
- net at D1.1 (K): now also R6.1
- net at Q10.3 (D): now also R6.2
- net at D8.1 (K), D9.1 (K): now also C36.1, S6.1, S6.2; no longer C19.1
- net at IC1.5 (PH0): now also Y2.3
- net at U4.12 (P01/XL2), Y1.2: now also C22.1; no longer C23.1
- removed net +3.3VA: C31.1, C35.1, IC1.13 (VDDA)
- removed net AGND: C1.2, C10.2, C11.2, C12.2, C13.2, C14.2, C15.2, C16.2, C17.2, C18.2, C2.2, C20.2, C21.2, C44.2, C5.2, C6.2, C7.2, C9.2, NT2.2, R1.1, R2.1, R3.1, R4.1, U1.8 (GND), U10.2 (GND), U3.2 (GND), U7.6 (GND)
- removed net BATT_NET: C36.1, S2.2, U9.11 (VCC), U9.2 (VCC), U9.3 (VCC), U9.9 (EN)
- new net +3V3: C1.1, C11.1, C18.1, C21.2, C27.2, C28.2, C29.2, C30.1, C32.2, C43.1, C6.1, C7.1, C8.2, IC1.1 (VBAT), IC1.19 (VDD_1), IC1.32 (VDD_2), IC1.48 (VDD_3), IC1.64 (VDD_4), M1.3 (Pin_3), M2.3 (Pin_3), R10.1, R11.1, R12.2, R16.1, R19.2, R20.2, R21.2, R23.1, R25.2, R26.2, R28.1, R9.1, U1.5 (VDDIO), U3.1 (IN), U3.3 (EN), U4.16 (VDD), U5.6 (VOUT), U7.5 (VDDIO), U8.5 (OUT), Y2.4
- no-connect marks 11 -> 26
Other:
- note added: "Diode check turnon voltage forward and make sure its below voltage threshold for reset"
- note added: "Self rsonsane frequency for capacitors for ripple rejecgion"
- note added: "check polarity of reset Y wehther SWD host floats or pulls up on no reset"
- note added: "pulldowns for en"
- note added: "vdd 3v3a ADD PULLUP FOR SPI vddio 3v3"
- note removed: "* 2 footprint options"
- note removed: "Mounting holes"
- moved on the sheet: C12, C7

Commit message: rev2 done !
Parts:
- removed C36: 0.1uF, Capacitor_SMD:C_0603_1608Metric_Pad1.08x0.95mm_HandSolder, symbol Device:C
- removed R10, R16: 10k, Resistor_SMD:R_0603_1608Metric_Pad0.98x0.95mm_HandSolder, symbol Device:R
- removed SK1, SK2, SK3, SK4: M2, MountingHole:MountingHole_2.2mm_M2, symbol bloo-rescue:MountingHole-Mechanical-mouse_v2-rescue
- removed TP7: V_EXT_TP, Connector_PinHeader_2.54mm:PinHeader_1x01_P2.54mm_Vertical, symbol Connector:TestPoint
- added C38, C40: 0.1uF, Capacitor_SMD:C_0603_1608Metric_Pad1.08x0.95mm_HandSolder, symbol Device:C
- IC1: footprint QFP50P1200X1200X160-64N -> STM32F405RGT6:QFP50P1200X1200X160-64N
- renumbered S2 to PWR1, S6 to RST1, S4 to S1, S3 to S2, S1 to S3
Connections:
- net +3V3: now also M1.4 (Pin_4), M2.4 (Pin_4); no longer M1.3 (Pin_3), M2.3 (Pin_3)
- net BC_RST: now also C38.1
- net GND: now also M1.1 (Pin_1), M2.1 (Pin_1), C38.2, C40.2; no longer M1.6 (Pin_6), M2.6 (Pin_6)
- net M1_ENC_A: now also M1.3 (Pin_3); no longer M2.4 (Pin_4)
- net M1_ENC_B: now also M1.2 (Pin_2); no longer M2.5 (Pin_5)
- net M1_OUT_1: now also M1.6 (Pin_6); no longer M2.1 (Pin_1)
- net M1_OUT_2: now also M1.5 (Pin_5); no longer M2.2 (Pin_2)
- net M2_ENC_A: now also M2.3 (Pin_3); no longer M1.4 (Pin_4)
- net M2_ENC_B: now also M2.2 (Pin_2); no longer M1.5 (Pin_5)
- net M2_OUT_1: now also M2.6 (Pin_6); no longer M1.1 (Pin_1)
- net M2_OUT_2: now also M2.5 (Pin_5); no longer M1.2 (Pin_2)
- net RST: now also C40.1
- no-connect marks 26 -> 27
Other:
- note removed: "* Resistors here act as current limiting resistors. Check that the resistor value properly limits current. Check the bluepills current limit for gpio"
- note removed: "Diode check turnon voltage forward and make sure its below voltage threshold for reset"
- note removed: "Self rsonsane frequency for capacitors for ripple rejecgion"
- note removed: "Skates"
- note removed: "check polarity of reset Y wehther SWD host floats or pulls up on no reset"
- note removed: "vdd 3v3a ADD PULLUP FOR SPI vddio 3v3"

Commit message: Micromouse is assembled and turns on! LEDs work as well. IOC is updated.
Parts:
- C1, C10, C11, C12, C13, C14, C15, C16, C17, C18, C19, C2, C20, C21, C22, C23, C24, C25, C26, C27, C28, C29, C3, C30, C31, C32, C33, C34, C35, C37, C38, C39, C4, C40, C41, C42, C43, C44, C5, C6, C7, C8, C9, D10, D4, D5, D6, D7, D8, D9, L2, M1, M2, Q10, Q11, Q12, Q9, R1, R11, R12, R13, R14, R15, R17, R18, R19, R2, R20, R21, R22, R23, R24, R25, R26, R27, R28, R3, R4, R5, R6, R7, R8, R9, RST1, S1, S2, S3, U10, U11, U3, U4, U5, U7, U8, U9, Y1, Y2: now not fitted
Connections:
- net IMU_INT: no longer names the net of U7.4 (INT1/INT)
- no-connect marks 27 -> 54
Other:
- note added: "Note buttons are now: https://www.digikey.com/en/products/detail/same-sky-formerly-cui-devices/TS20-42-25-WT-160-SMT-TR/16590894"
